Commit message: cubos flacos

File: src/sawyer_simulator/sawyer_sim_examples/models/block/blue_cube.urdf (robot description, URDF)
Before this commit: robot blue_cube, 1 links, 0 joints
Links:
- link base_link: geometry collision box size=0.075 0.04 0.05; visual box size=0.075 0.04 0.05

File: src/sawyer_simulator/sawyer_sim_examples/models/block/green_cube.urdf (robot description, URDF)
Before this commit: robot green_cube, 1 links, 0 joints
Links:
- link base_link: geometry collision box size=0.075 0.04 0.05; visual box size=0.075 0.04 0.05

File: src/sawyer_simulator/sawyer_sim_examples/models/block/red_cube.urdf (robot description, URDF)
Before this commit: robot red_cube, 1 links, 0 joints
Links:
- link base_link: geometry collision box size=0.075 0.04 0.05; visual box size=0.075 0.04 0.05
