Commit message: add open gripper and close gripper

File: src/sawyer_robot/sawyer_description/urdf/banda.xacro (robot description, xacro)
@@ -5,5 +5,5 @@
         <parent link="world"/>
         <child link="belt_visual"/>
-        <origin xyz="0.5 -1.0 -0.91488" rpy="0 0 1.57"/> <!-- Rotación en Z -->
+        <origin xyz="0.3 -0.9 -0.91488" rpy="0 0 1.57"/> <!-- Rotación en Z -->
     </joint>
     <!-- Definición de la banda visual -->

Commit message: Añadir nueva funcionalidad en la rama feature-nueva-funcionalidad

File: src/sawyer_robot/sawyer_description/urdf/banda.xacro (robot description, xacro)
@@ -12,5 +12,6 @@
             <origin xyz="-1.1327e-16 -3.3286e-17 0.66619" rpy="0 0 0"/>
             <mass value="71.955"/>
-            <inertia ixx="7.5972" ixy="-1.3948e-14" ixz="-1.9328e-17" iyy="0.99673" iyz="-9.2056e-18" izz="8.1168"/>
+            <inertia ixx="7.5972" ixy="-1.3948e-14" ixz="-1.9328e-17"
+                     iyy="0.99673" iyz="-9.2056e-18" izz="8.1168"/>
         </inertial>
         <visual>
@@ -43,5 +44,6 @@
             <origin xyz="0 0 0" rpy="0 0 0"/>
             <mass value="100"/>
-            <inertia ixx="0.0" ixy="0.0" ixz="0.0" iyy="0.0" iyz="0.0" izz="0.0"/>
+            <inertia ixx="0.0" ixy="0.0" ixz="0.0"
+                     iyy="0.0" iyz="0.0" izz="0.0"/>
         </inertial>
         <visual>
@@ -60,4 +62,31 @@
             </geometry>
         </collision>
+        <!-- Cámara binaria para detección de objetos -->
+        <gazebo reference="belt_moving">
+            <sensor type="camera" name="binary_camera">
+                <update_rate>30</update_rate>
+                <camera>
+                    <horizontal_fov>1.047</horizontal_fov>
+                    <image>
+                        <width>640</width>
+                        <height>480</height>
+                        <format>L8</format>  <!-- Imagen en escala de grises (binaria) -->
+                    </image>
+                    <clip>
+                        <near>0.1</near>
+                        <far>5.0</far>
+                    </clip>
+                    <pose>0 0 0.5 0 0 0</pose>  <!-- Cámara encima de la banda -->
+                </camera>
+                <plugin name="camera_plugin" filename="libgazebo_ros_camera.so">
+                    <always_on>true</always_on>
+                    <update_rate>30.0</update_rate>
+                    <camera_name>binary_camera</camera_name>
+                    <image_topic_name>/camera/image_raw</image_topic_name>
+                    <info_topic_name>/camera/camera_info</info_topic_name>
+                    <frame_name>camera_link</frame_name>
+                </plugin>
+            </sensor>
+        </gazebo>
     </link>
     <!-- Plugin para el movimiento de la banda -->

Commit message: Opencv

File: src/sawyer_robot/sawyer_description/urdf/banda.xacro (robot description, xacro)
@@ -61,4 +61,85 @@
         </collision>
     </link>
+    <!-- Nuevo bloque: Soporte de la cámara -->
+    <link name="camera_mount">
+        <inertial>
+            <mass value="1.0"/>
+            <origin xyz="0 0 0"/>
+            <inertia ixx="0.1" ixy="0.0" ixz="0.0" iyy="0.1" iyz="0.0" izz="0.1"/>
+        </inertial>
+        <visual>
+            <geometry>
+                <box size="0.4 0.4 0.1"/> <!-- Tamaño del bloque -->
+            </geometry>
+            <material name="gray">
+                <color rgba="0.5 0.5 0.5 1.0"/> <!-- Color gris -->
+            </material>
+        </visual>
+        <collision>
+            <geometry>
+                <box size="0.4 0.4 0.1"/>
+            </geometry>
+        </collision>
+    </link>
+    <!-- Joint para fijar la cámara sobre la banda -->
+    <joint name="camera_mount_joint" type="fixed">
+        <parent link="belt_visual"/>  <!-- Fijado a la banda transportadora -->
+        <child link="camera_mount"/>
+        <origin xyz="0 0 1.5" rpy="0 0 0"/> <!-- Ajusta la altura si es necesario -->
+    </joint>
+    <!-- Cámara RGB montada en el bloque -->
+    <link name="camera_rgb">
+        <inertial>
+            <mass value="0.5"/>
+            <origin xyz="0 0 0"/>
+            <inertia ixx="0.01" ixy="0.0" ixz="0.0" iyy="0.01" iyz="0.0" izz="0.01"/>
+        </inertial>
+        <visual>
+            <origin xyz="0 0 0" rpy="0 0 0"/>
+            <geometry>
+                <box size="0.1 0.1 0.05"/>  <!-- Simulación de la cámara -->
+            </geometry>
+            <material name="black">
+                <color rgba="0 0 0 1"/>
+            </material>
+        </visual>
+        <collision>
+            <geometry>
+                <box size="0.1 0.1 0.05"/>
+            </geometry>
+        </collision>
+    </link>
+    <!-- Joint para montar la cámara en el bloque y orientarla hacia abajo -->
+    <joint name="camera_rgb_joint" type="fixed">
+        <parent link="camera_mount"/>
+        <child link="camera_rgb"/>
+        <origin xyz="0 0 0.05" rpy="0 1.57 0"/> <!-- Rotación para mirar hacia abajo -->
+    </joint>
+    <!-- Configuración de la cámara en Gazebo -->
+    <gazebo reference="camera_rgb">
+        <sensor name="camera_sensor" type="camera">
+            <update_rate>30</update_rate>
+            <camera>
+                <horizontal_fov>1.047</horizontal_fov> <!-- 60 grados -->
+                <image>
+                    <width>640</width>
+                    <height>480</height>
+                    <format>R8G8B8</format>
+                </image>
+                <clip>
+                    <near>0.1</near>
+                    <far>10.0</far>
+                </clip>
+            </camera>
+            <plugin name="camera_plugin" filename="libgazebo_ros_camera.so">
+                <alwaysOn>true</alwaysOn>
+                <updateRate>30</updateRate>
+                <cameraName>camera_rgb</cameraName>
+                <imageTopicName>/camera/image_raw</imageTopicName>
+                <cameraInfoTopicName>/camera/camera_info</cameraInfoTopicName>
+                <frameName>camera_rgb</frameName>
+            </plugin>
+        </sensor>
+    </gazebo>
     <!-- Plugin para el movimiento de la banda -->
     <gazebo>
